File: kicad/pico_parrot/pico_parrot.kicad_sch (KiCad schematic)
At the start: 37 parts, among them J1 AudioJack3_BaofengMicPort, J2 AudioJack3_BaofengSpeaker, Q1 2N3904, Q2 MMBT3904, U1 Pico, U2 AMS1117-5.0

Commit message: parrot
Parts:
- added C13, C14, C16, C18: 10uF, Capacitor_THT:C_Disc_D4.3mm_W1.9mm_P5.00mm, symbol Device:C
- added C15, C17: 100nF, Capacitor_THT:C_Disc_D4.3mm_W1.9mm_P5.00mm, symbol Device:C
- J_baofeng_2.5mm: renamed from J2; footprint (none) -> footprints:PJ-307_Modded
- J_baofeng_3.5mm: renamed from J1; footprint (none) -> footprints:PJ-307_Modded
- TP2: value TestPointGND -> GND
- U1: footprint RPi_Pico:RPi_Pico_SMD_TH -> MCU_RaspberryPi_and_Boards:RPi_Pico_SMD_TH
- renumbered TP3 to 3.3V, TP1 to VCC
Connections:
- net +3.3V: now also C17.1, C18.1
- net GND: now also C13.2, C14.2, C15.2, C16.2, C17.2, C18.2
- net at C6.2, C8.2, U1.39 (VSYS)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: now also C15.1, C16.1
- net at C10.1, C9.1, U2.3 (VI)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: now also C13.1, C14.1
